Commit message: feat: support three AGV models and reliable controls

File: src/agv_description/urdf/agv.urdf.xacro (robot description, xacro)
@@ -3,9 +3,9 @@
   <xacro:property name="wheel_radius" value="0.10"/><xacro:property name="wheel_width" value="0.05"/>
   <link name="base_footprint"/>
-  <link name="base_link"><visual><geometry><box size="1.2 0.8 0.35"/></geometry><material name="blue"><color rgba="0.1 0.3 0.8 1"/></material></visual><collision><geometry><box size="1.2 0.8 0.35"/></geometry></collision><inertial><mass value="120"/><origin xyz="0 0 0"/><inertia ixx="8" ixy="0" ixz="0" iyy="15" iyz="0" izz="20"/></inertial></link>
+  <link name="base_link"><visual><geometry><box size="1.2 0.8 0.35"/></geometry><material name="blue"><color rgba="0.1 0.3 0.8 1"/></material></visual><collision><origin xyz="0 0 0.05"/><geometry><box size="1.2 0.8 0.25"/></geometry></collision><inertial><mass value="1163.5"/><origin xyz="0 0 0"/><inertia ixx="73.94" ixy="0" ixz="0" iyy="151.52" iyz="0" izz="201.67"/></inertial></link>
   <joint name="base_footprint_joint" type="fixed"><parent link="base_footprint"/><child link="base_link"/><origin xyz="0 0 0.275"/></joint>
   <xacro:macro name="module" params="id x y">
     <link name="module_${id}_carrier"><visual><geometry><cylinder radius="0.11" length="0.08"/></geometry></visual><collision><geometry><cylinder radius="0.11" length="0.08"/></geometry></collision><inertial><mass value="5"/><inertia ixx="0.03" ixy="0" ixz="0" iyy="0.03" iyz="0" izz="0.04"/></inertial></link>
-    <joint name="module_${id}_steering_joint" type="continuous"><parent link="base_link"/><child link="module_${id}_carrier"/><origin xyz="${x} ${y} -0.175"/><axis xyz="0 0 1"/><dynamics damping="0.2" friction="0.05"/></joint>
+    <joint name="module_${id}_steering_joint" type="continuous"><parent link="base_link"/><child link="module_${id}_carrier"/><origin xyz="${x} ${y} -0.175"/><axis xyz="0 0 1"/><dynamics damping="1.0" friction="0.05"/></joint>
     <xacro:wheel id="${id}" side="left" offset="0.05" axis="1"/><xacro:wheel id="${id}" side="right" offset="-0.05" axis="-1"/>
   </xacro:macro>

Commit message: Fix differential swerve simulation stability

File: src/agv_description/urdf/agv.urdf.xacro (robot description, xacro)
@@ -11,7 +11,7 @@
   </xacro:macro>
   <xacro:macro name="wheel" params="id side offset axis">
-    <link name="module_${id}_${side}_wheel"><visual><origin rpy="1.5708 0 0"/><geometry><cylinder radius="${wheel_radius}" length="${wheel_width}"/></geometry></visual><collision><origin rpy="1.5708 0 0"/><geometry><cylinder radius="${wheel_radius}" length="${wheel_width}"/></geometry></collision><inertial><mass value="2"/><inertia ixx="0.01" ixy="0" ixz="0" iyy="0.005" iyz="0" izz="0.01"/></inertial></link>
-    <joint name="module_${id}_${side}_wheel_joint" type="continuous"><parent link="module_${id}_carrier"/><child link="module_${id}_${side}_wheel"/><origin xyz="0 ${offset} -0.10"/><axis xyz="0 ${axis} 0"/><dynamics damping="0.05"/></joint>
-    <gazebo reference="module_${id}_${side}_wheel"><mu1>1.5</mu1><mu2>1.5</mu2></gazebo>
+    <link name="module_${id}_${side}_wheel"><visual><geometry><cylinder radius="${wheel_radius}" length="${wheel_width}"/></geometry></visual><collision><geometry><cylinder radius="${wheel_radius}" length="${wheel_width}"/></geometry></collision><inertial><mass value="2"/><inertia ixx="0.005416666666666667" ixy="0" ixz="0" iyy="0.005416666666666667" iyz="0" izz="0.01"/></inertial></link>
+    <joint name="module_${id}_${side}_wheel_joint" type="continuous"><parent link="module_${id}_carrier"/><child link="module_${id}_${side}_wheel"/><origin xyz="0 ${offset} -0.10" rpy="${-axis*pi/2} 0 0"/><axis xyz="0 0 1"/><dynamics damping="0.05"/></joint>
+    <gazebo reference="module_${id}_${side}_wheel"><mu1>1.3</mu1><mu2>1.3</mu2><kp>500000.0</kp><kd>10.0</kd><maxVel>0.1</maxVel><minDepth>0.001</minDepth></gazebo>
   </xacro:macro>
   <xacro:module id="1" x="0.45" y="0.325"/><xacro:module id="2" x="0.45" y="-0.325"/><xacro:module id="3" x="-0.45" y="-0.325"/><xacro:module id="4" x="-0.45" y="0.325"/>

Commit message: Add Nav2 localization and omnidirectional navigation

File: src/agv_description/urdf/agv.urdf.xacro (robot description, xacro)
@@ -3,5 +3,5 @@
   <xacro:property name="wheel_radius" value="0.10"/><xacro:property name="wheel_width" value="0.05"/>
   <link name="base_footprint"/>
-  <link name="base_link"><visual><geometry><box size="1.2 0.8 0.35"/></geometry><material name="blue"><color rgba="0.1 0.3 0.8 1"/></material></visual><collision><origin xyz="0 0 0.05"/><geometry><box size="1.2 0.8 0.25"/></geometry></collision><inertial><mass value="1163.5"/><origin xyz="0 0 0"/><inertia ixx="73.94" ixy="0" ixz="0" iyy="151.52" iyz="0" izz="201.67"/></inertial></link>
+  <link name="base_link"><visual><geometry><box size="1.2 0.8 0.35"/></geometry><material name="blue"><color rgba="0.1 0.3 0.8 1"/></material></visual><collision><origin xyz="0 0 0.05"/><geometry><box size="1.2 0.8 0.25"/></geometry></collision><inertial><mass value="60.0"/><origin xyz="0 0 0"/><inertia ixx="3.8125" ixy="0" ixz="0" iyy="7.8125" iyz="0" izz="10.4"/></inertial></link>
   <joint name="base_footprint_joint" type="fixed"><parent link="base_footprint"/><child link="base_link"/><origin xyz="0 0 0.275"/></joint>
   <xacro:macro name="module" params="id x y">
